Commit message: replace package:// with () in mesh stl file

File: src/jetrover_description/urdf/arm.urdf.xacro (robot description, xacro)
@@ -24,5 +24,5 @@
       <geometry>
         <mesh
-          filename="package://jetrover_description/meshes/arm/link1.STL" />
+          filename="$(find jetrover_description)/meshes/arm/link1.STL" />
       </geometry>
       <material name="green"/>
@@ -34,5 +34,5 @@
       <geometry>
         <mesh
-          filename="package://jetrover_description/meshes/arm/link1.STL" />
+          filename="$(find jetrover_description)/meshes/arm/link1.STL" />
       </geometry>
     </collision>
@@ -60,5 +60,5 @@
       <geometry>
         <mesh
-          filename="package://jetrover_description/meshes/arm/servo_link1.STL" />
+          filename="$(find jetrover_description)/meshes/arm/servo_link1.STL" />
       </geometry>
       <material name="black"/>
@@ -70,5 +70,5 @@
       <geometry>
         <mesh
-          filename="package://jetrover_description/meshes/arm/servo_link1_collision.stl" />
+          filename="$(find jetrover_description)/meshes/arm/servo_link1_collision.stl" />
       </geometry>
     </collision>
@@ -109,5 +109,5 @@
       <geometry>
         <mesh
-          filename="package://jetrover_description/meshes/arm/link2.STL" />
+          filename="$(find jetrover_description)/meshes/arm/link2.STL" />
       </geometry>
       <material name="green"/>
@@ -119,5 +119,5 @@
       <geometry>
         <mesh
-          filename="package://jetrover_description/meshes/arm/link2_collision.stl" />
+          filename="$(find jetrover_description)/meshes/arm/link2_collision.stl" />
       </geometry>
     </collision>
@@ -163,5 +163,5 @@
       <geometry>
         <mesh
-          filename="package://jetrover_description/meshes/arm/link3.STL" />
+          filename="$(find jetrover_description)/meshes/arm/link3.STL" />
       </geometry>
       <material name="green"/>
@@ -173,5 +173,5 @@
       <geometry>
         <mesh
-          filename="package://jetrover_description/meshes/arm/link3_collision.stl" />
+          filename="$(find jetrover_description)/meshes/arm/link3_collision.stl" />
       </geometry>
     </collision>
@@ -217,5 +217,5 @@
       <geometry>
         <mesh
-          filename="package://jetrover_description/meshes/arm/link4.STL" />
+          filename="$(find jetrover_description)/meshes/arm/link4.STL" />
       </geometry>
       <material name="green"/>
@@ -227,5 +227,5 @@
       <geometry>
         <mesh
-          filename="package://jetrover_description/meshes/arm/link4_collision.stl" />
+          filename="$(find jetrover_description)/meshes/arm/link4_collision.stl" />
       </geometry>
     </collision>
@@ -271,5 +271,5 @@
       <geometry>
         <mesh
-          filename="package://jetrover_description/meshes/arm/servo_link2.STL" />
+          filename="$(find jetrover_description)/meshes/arm/servo_link2.STL" />
       </geometry>
       <material name="black"/>
@@ -281,5 +281,5 @@
       <geometry>
         <mesh
-          filename="package://jetrover_description/meshes/arm/servo_link2_collision.stl" />
+          filename="$(find jetrover_description)/meshes/arm/servo_link2_collision.stl" />
       </geometry>
     </collision>
@@ -320,5 +320,5 @@
       <geometry>
         <mesh
-          filename="package://jetrover_description/meshes/arm/link5.STL" />
+          filename="$(find jetrover_description)/meshes/arm/link5.STL" />
       </geometry>
       <material name="black"/>
@@ -330,5 +330,5 @@
       <geometry>
         <mesh
-          filename="package://jetrover_description/meshes/arm/link5.STL" />
+          filename="$(find jetrover_description)/meshes/arm/link5.STL" />
       </geometry>
     </collision>
@@ -374,5 +374,5 @@
       <geometry>
         <mesh
-          filename="package://jetrover_description/meshes/arm/gripper_link.STL" />
+          filename="$(find jetrover_description)/meshes/arm/gripper_link.STL" />
       </geometry>
       <material name="black"/>
@@ -384,5 +384,5 @@
       <geometry>
         <mesh
-          filename="package://jetrover_description/meshes/arm/gripper_link_collision.stl" />
+          filename="$(find jetrover_description)/meshes/arm/gripper_link_collision.stl" />
       </geometry>
     </collision>

File: src/jetrover_description/urdf/car_acker.urdf.xacro (robot description, xacro)
@@ -35,15 +35,15 @@
       <geometry>
         <mesh
-          filename="package://jetrover_description/meshes/acker/base_link.stl" />
-      </geometry>
-      <material name="black"/>
-    </visual>
-    <collision>
-      <origin
-        xyz="0 0 0"
-        rpy="0 0 0" />
-      <geometry>
-        <mesh
-          filename="package://jetrover_description/meshes/acker/base_link.stl" />
+          filename="$(find jetrover_description)/meshes/acker/base_link.stl" />
+      </geometry>
+      <material name="black"/>
+    </visual>
+    <collision>
+      <origin
+        xyz="0 0 0"
+        rpy="0 0 0" />
+      <geometry>
+        <mesh
+          filename="$(find jetrover_description)/meshes/acker/base_link.stl" />
       </geometry>
     </collision>
@@ -71,5 +71,5 @@
       <geometry>
         <mesh
-          filename="package://jetrover_description/meshes/acker/base_green_link.stl" />
+          filename="$(find jetrover_description)/meshes/acker/base_green_link.stl" />
       </geometry>
       <material name="green"/>
@@ -81,5 +81,5 @@
       <geometry>
         <mesh
-          filename="package://jetrover_description/meshes/acker/base_green_link.stl" />
+          filename="$(find jetrover_description)/meshes/acker/base_green_link.stl" />
       </geometry>
     </collision>
@@ -120,15 +120,15 @@
       <geometry>
         <mesh
-          filename="package://jetrover_description/meshes/acker/wheel_left_front_link.stl" />
-      </geometry>
-      <material name="black"/>
-    </visual>
-    <collision>
-      <origin
-        xyz="0 0 0"
-        rpy="0 0 0" />
-      <geometry>
-        <mesh
-          filename="package://jetrover_description/meshes/acker/wheel_left_front_link.stl" />
+          filename="$(find jetrover_description)/meshes/acker/wheel_left_front_link.stl" />
+      </geometry>
+      <material name="black"/>
+    </visual>
+    <collision>
+      <origin
+        xyz="0 0 0"
+        rpy="0 0 0" />
+      <geometry>
+        <mesh
+          filename="$(find jetrover_description)/meshes/acker/wheel_left_front_link.stl" />
       </geometry>
     </collision>
@@ -169,15 +169,15 @@
       <geometry>
         <mesh
-          filename="package://jetrover_description/meshes/acker/wheel_left_back_link.stl" />
-      </geometry>
-      <material name="black"/>
-    </visual>
-    <collision>
-      <origin
-        xyz="0 0 0"
-        rpy="0 0 0" />
-      <geometry>
-        <mesh
-          filename="package://jetrover_description/meshes/acker/wheel_left_back_link.stl" />
+          filename="$(find jetrover_description)/meshes/acker/wheel_left_back_link.stl" />
+      </geometry>
+      <material name="black"/>
+    </visual>
+    <collision>
+      <origin
+        xyz="0 0 0"
+        rpy="0 0 0" />
+      <geometry>
+        <mesh
+          filename="$(find jetrover_description)/meshes/acker/wheel_left_back_link.stl" />
       </geometry>
     </collision>
@@ -218,15 +218,15 @@
       <geometry>
         <mesh
-          filename="package://jetrover_description/meshes/acker/wheel_right_front_link.stl" />
-      </geometry>
-      <material name="black"/>
-    </visual>
-    <collision>
-      <origin
-        xyz="0 0 0"
-        rpy="0 0 0" />
-      <geometry>
-        <mesh
-          filename="package://jetrover_description/meshes/acker/wheel_right_front_link.stl" />
+          filename="$(find jetrover_description)/meshes/acker/wheel_right_front_link.stl" />
+      </geometry>
+      <material name="black"/>
+    </visual>
+    <collision>
+      <origin
+        xyz="0 0 0"
+        rpy="0 0 0" />
+      <geometry>
+        <mesh
+          filename="$(find jetrover_description)/meshes/acker/wheel_right_front_link.stl" />
       </geometry>
     </collision>
@@ -267,15 +267,15 @@
       <geometry>
         <mesh
-          filename="package://jetrover_description/meshes/acker/wheel_right_back_link.stl" />
-      </geometry>
-      <material name="black"/>
-    </visual>
-    <collision>
-      <origin
-        xyz="0 0 0"
-        rpy="0 0 0" />
-      <geometry>
-        <mesh
-          filename="package://jetrover_description/meshes/acker/wheel_right_back_link.stl" />
+          filename="$(find jetrover_description)/meshes/acker/wheel_right_back_link.stl" />
+      </geometry>
+      <material name="black"/>
+    </visual>
+    <collision>
+      <origin
+        xyz="0 0 0"
+        rpy="0 0 0" />
+      <geometry>
+        <mesh
+          filename="$(find jetrover_description)/meshes/acker/wheel_right_back_link.stl" />
       </geometry>
     </collision>

File: src/jetrover_description/urdf/car_mecanum.urdf.xacro (robot description, xacro)
@@ -21,5 +21,5 @@
       <geometry>
         <mesh
-          filename="package://jetrover_description/meshes/mecanum/base_link.stl" />
+          filename="$(find jetrover_description)/meshes/mecanum/base_link.stl" />
       </geometry>
       <material name="green"/>
@@ -31,5 +31,5 @@
       <geometry>
         <mesh
-          filename="package://jetrover_description/meshes/mecanum/base_link_collision.stl" />
+          filename="$(find jetrover_description)/meshes/mecanum/base_link_collision.stl" />
       </geometry>
     </collision>
@@ -57,15 +57,15 @@
       <geometry>
         <mesh
-          filename="package://jetrover_description/meshes/mecanum/wheel_left_front_link.stl" />
-      </geometry>
-      <material name="black"/>
-    </visual>
-    <collision>
-      <origin
-        xyz="0 0 0"
-        rpy="0 0 0" />
-      <geometry>
-        <mesh
-          filename="package://jetrover_description/meshes/mecanum/wheel_left_front_link_collision.stl" />
+          filename="$(find jetrover_description)/meshes/mecanum/wheel_left_front_link.stl" />
+      </geometry>
+      <material name="black"/>
+    </visual>
+    <collision>
+      <origin
+        xyz="0 0 0"
+        rpy="0 0 0" />
+      <geometry>
+        <mesh
+          filename="$(find jetrover_description)/meshes/mecanum/wheel_left_front_link_collision.stl" />
       </geometry>
     </collision>
@@ -106,15 +106,15 @@
       <geometry>
         <mesh
-          filename="package://jetrover_description/meshes/mecanum/wheel_left_back_link.stl" />
-      </geometry>
-      <material name="black"/>
-    </visual>
-    <collision>
-      <origin
-        xyz="0 0 0"
-        rpy="0 0 0" />
-      <geometry>
-        <mesh
-          filename="package://jetrover_description/meshes/mecanum/wheel_left_back_link_collision.stl" />
+          filename="$(find jetrover_description)/meshes/mecanum/wheel_left_back_link.stl" />
+      </geometry>
+      <material name="black"/>
+    </visual>
+    <collision>
+      <origin
+        xyz="0 0 0"
+        rpy="0 0 0" />
+      <geometry>
+        <mesh
+          filename="$(find jetrover_description)/meshes/mecanum/wheel_left_back_link_collision.stl" />
       </geometry>
     </collision>
@@ -155,15 +155,15 @@
       <geometry>
         <mesh
-          filename="package://jetrover_description/meshes/mecanum/wheel_right_front_link.stl" />
-      </geometry>
-      <material name="black"/>
-    </visual>
-    <collision>
-      <origin
-        xyz="0 0 0"
-        rpy="0 0 0" />
-      <geometry>
-        <mesh
-            filename="package://jetrover_description/meshes/mecanum/wheel_right_front_link_collision.stl" />
+          filename="$(find jetrover_description)/meshes/mecanum/wheel_right_front_link.stl" />
+      </geometry>
+      <material name="black"/>
+    </visual>
+    <collision>
+      <origin
+        xyz="0 0 0"
+        rpy="0 0 0" />
+      <geometry>
+        <mesh
+            filename="$(find jetrover_description)/meshes/mecanum/wheel_right_front_link_collision.stl" />
       </geometry>
     </collision>
@@ -204,15 +204,15 @@
       <geometry>
         <mesh
-          filename="package://jetrover_description/meshes/mecanum/wheel_right_back_link.stl" />
-      </geometry>
-      <material name="black"/>
-    </visual>
-    <collision>
-      <origin
-        xyz="0 0 0"
-        rpy="0 0 0" />
-      <geometry>
-        <mesh
-            filename="package://jetrover_description/meshes/mecanum/wheel_right_back_link_collision.stl" />
+          filename="$(find jetrover_description)/meshes/mecanum/wheel_right_back_link.stl" />
+      </geometry>
+      <material name="black"/>
+    </visual>
+    <collision>
+      <origin
+        xyz="0 0 0"
+        rpy="0 0 0" />
+      <geometry>
+        <mesh
+            filename="$(find jetrover_description)/meshes/mecanum/wheel_right_back_link_collision.stl" />
       </geometry>
     </collision>

File: src/jetrover_description/urdf/car_tank.urdf.xacro (robot description, xacro)
@@ -21,5 +21,5 @@
       <geometry>
         <mesh
-          filename="package://jetrover_description/meshes/tank/base_link.stl" />
+          filename="$(find jetrover_description)/meshes/tank/base_link.stl" />
       </geometry>
       <material name="green"/>
@@ -31,5 +31,5 @@
       <geometry>
         <mesh
-          filename="package://jetrover_description/meshes/tank/base_link.stl" />
+          filename="$(find jetrover_description)/meshes/tank/base_link.stl" />
       </geometry>
     </collision>
@@ -57,5 +57,5 @@
       <geometry>
         <mesh
-          filename="package://jetrover_description/meshes/tank/wheel_link.stl" />
+          filename="$(find jetrover_description)/meshes/tank/wheel_link.stl" />
       </geometry>
       <material name="black"/>
@@ -67,5 +67,5 @@
       <geometry>
         <mesh
-          filename="package://jetrover_description/meshes/tank/wheel_link.stl" />
+          filename="$(find jetrover_description)/meshes/tank/wheel_link.stl" />
       </geometry>
     </collision>

File: src/jetrover_description/urdf/common.urdf.xacro (robot description, xacro)
@@ -23,5 +23,5 @@
       <geometry>
         <mesh
-          filename="package://jetrover_description/meshes/common/back_shell_black_link.stl" />
+          filename="$(find jetrover_description)/meshes/common/back_shell_black_link.stl" />
       </geometry>
       <material name="black"/>
@@ -33,5 +33,5 @@
       <geometry>
         <mesh
-          filename="package://jetrover_description/meshes/common/back_shell_black_link_collision.stl" />
+          filename="$(find jetrover_description)/meshes/common/back_shell_black_link_collision.stl" />
       </geometry>
     </collision>
@@ -72,5 +72,5 @@
       <geometry>
         <mesh
-          filename="package://jetrover_description/meshes/common/back_shell_green_link.stl" />
+          filename="$(find jetrover_description)/meshes/common/back_shell_green_link.stl" />
       </geometry>
       <material name="green"/>
@@ -82,5 +82,5 @@
       <geometry>
         <mesh
-          filename="package://jetrover_description/meshes/common/back_shell_green_link_collision.stl" />
+          filename="$(find jetrover_description)/meshes/common/back_shell_green_link_collision.stl" />
       </geometry>
     </collision>

File: src/jetrover_description/urdf/depth_camera.urdf.xacro (robot description, xacro)
@@ -24,5 +24,5 @@
       <geometry>
         <mesh
-          filename="package://jetrover_description/meshes/arm/camera_connect_link.STL" />
+          filename="$(find jetrover_description)/meshes/arm/camera_connect_link.STL" />
       </geometry>
       <material name="black"/>
@@ -34,5 +34,5 @@
       <geometry>
         <mesh
-          filename="package://jetrover_description/meshes/arm/camera_connect_link.STL" />
+          filename="$(find jetrover_description)/meshes/arm/camera_connect_link.STL" />
       </geometry>
     </collision>
@@ -73,5 +73,5 @@
       <geometry>
         <mesh
-          filename="package://jetrover_description/meshes/arm/depth_cam_link.STL" />
+          filename="$(find jetrover_description)/meshes/arm/depth_cam_link.STL" />
       </geometry>
       <material
@@ -87,5 +87,5 @@
       <geometry>
         <mesh
-          filename="package://jetrover_description/meshes/arm/depth_cam_link_collision.stl" />
+          filename="$(find jetrover_description)/meshes/arm/depth_cam_link_collision.stl" />
       </geometry>
     </collision>

File: src/jetrover_description/urdf/gripper.urdf.xacro (robot description, xacro)
@@ -24,15 +24,15 @@
       <geometry>
         <mesh
-          filename="package://jetrover_description/meshes/gripper/r_link.STL" />
-      </geometry>
-      <material name="black"/>
-    </visual>
-    <collision>
-      <origin
-        xyz="0 0 0"
-        rpy="0 0 0" />
-      <geometry>
-        <mesh
-          filename="package://jetrover_description/meshes/gripper/r_link.STL" />
+          filename="$(find jetrover_description)/meshes/gripper/r_link.STL" />
+      </geometry>
+      <material name="black"/>
+    </visual>
+    <collision>
+      <origin
+        xyz="0 0 0"
+        rpy="0 0 0" />
+      <geometry>
+        <mesh
+          filename="$(find jetrover_description)/meshes/gripper/r_link.STL" />
       </geometry>
     </collision>
@@ -78,15 +78,15 @@
       <geometry>
         <mesh
-          filename="package://jetrover_description/meshes/gripper/l_link.STL" />
-      </geometry>
-      <material name="black"/>
-    </visual>
-    <collision>
-      <origin
-        xyz="0 0 0"
-        rpy="0 0 0" />
-      <geometry>
-        <mesh
-          filename="package://jetrover_description/meshes/gripper/l_link.STL" />
+          filename="$(find jetrover_description)/meshes/gripper/l_link.STL" />
+      </geometry>
+      <material name="black"/>
+    </visual>
+    <collision>
+      <origin
+        xyz="0 0 0"
+        rpy="0 0 0" />
+      <geometry>
+        <mesh
+          filename="$(find jetrover_description)/meshes/gripper/l_link.STL" />
       </geometry>
     </collision>
@@ -136,15 +136,15 @@
       <geometry>
         <mesh
-          filename="package://jetrover_description/meshes/gripper/l_in_link.STL" />
-      </geometry>
-      <material name="black"/>
-    </visual>
-    <collision>
-      <origin
-        xyz="0 0 0"
-        rpy="0 0 0" />
-      <geometry>
-        <mesh
-          filename="package://jetrover_description/meshes/gripper/l_in_link.STL" />
+          filename="$(find jetrover_description)/meshes/gripper/l_in_link.STL" />
+      </geometry>
+      <material name="black"/>
+    </visual>
+    <collision>
+      <origin
+        xyz="0 0 0"
+        rpy="0 0 0" />
+      <geometry>
+        <mesh
+          filename="$(find jetrover_description)/meshes/gripper/l_in_link.STL" />
       </geometry>
     </collision>
@@ -194,15 +194,15 @@
       <geometry>
         <mesh
-          filename="package://jetrover_description/meshes/gripper/l_out_link.STL" />
-      </geometry>
-      <material name="black"/>
-    </visual>
-    <collision>
-      <origin
-        xyz="0 0 0"
-        rpy="0 0 0" />
-      <geometry>
-        <mesh
-          filename="package://jetrover_description/meshes/gripper/l_out_link.STL" />
+          filename="$(find jetrover_description)/meshes/gripper/l_out_link.STL" />
+      </geometry>
+      <material name="black"/>
+    </visual>
+    <collision>
+      <origin
+        xyz="0 0 0"
+        rpy="0 0 0" />
+      <geometry>
+        <mesh
+          filename="$(find jetrover_description)/meshes/gripper/l_out_link.STL" />
       </geometry>
     </collision>
@@ -252,15 +252,15 @@
       <geometry>
         <mesh
-          filename="package://jetrover_description/meshes/gripper/r_in_link.STL" />
-      </geometry>
-      <material name="black"/>
-    </visual>
-    <collision>
-      <origin
-        xyz="0 0 0"
-        rpy="0 0 0" />
-      <geometry>
-        <mesh
-          filename="package://jetrover_description/meshes/gripper/r_in_link.STL" />
+          filename="$(find jetrover_description)/meshes/gripper/r_in_link.STL" />
+      </geometry>
+      <material name="black"/>
+    </visual>
+    <collision>
+      <origin
+        xyz="0 0 0"
+        rpy="0 0 0" />
+      <geometry>
+        <mesh
+          filename="$(find jetrover_description)/meshes/gripper/r_in_link.STL" />
       </geometry>
     </collision>
@@ -310,15 +310,15 @@
       <geometry>
         <mesh
-          filename="package://jetrover_description/meshes/gripper/r_out_link.STL" />
-      </geometry>
-      <material name="black"/>
-    </visual>
-    <collision>
-      <origin
-        xyz="0 0 0"
-        rpy="0 0 0" />
-      <geometry>
-        <mesh
-          filename="package://jetrover_description/meshes/gripper/r_out_link.STL" />
+          filename="$(find jetrover_description)/meshes/gripper/r_out_link.STL" />
+      </geometry>
+      <material name="black"/>
+    </visual>
+    <collision>
+      <origin
+        xyz="0 0 0"
+        rpy="0 0 0" />
+      <geometry>
+        <mesh
+          filename="$(find jetrover_description)/meshes/gripper/r_out_link.STL" />
       </geometry>
     </collision>

File: src/jetrover_description/urdf/imu.urdf.xacro (robot description, xacro)
@@ -24,5 +24,5 @@
       <geometry>
         <mesh
-          filename="package://jetrover_description/meshes/common/imu_link.stl" />
+          filename="$(find jetrover_description)/meshes/common/imu_link.stl" />
       </geometry>
       <material name="black"/>
@@ -34,5 +34,5 @@
       <geometry>
         <mesh
-          filename="package://jetrover_description/meshes/common/imu_link.stl" />
+          filename="$(find jetrover_description)/meshes/common/imu_link.stl" />
       </geometry>
     </collision>

File: src/jetrover_description/urdf/lidar.urdf.xacro (robot description, xacro)
@@ -24,5 +24,5 @@
       <geometry>
         <mesh
-          filename="package://jetrover_description/meshes/common/lidar_link.stl" />
+          filename="$(find jetrover_description)/meshes/common/lidar_link.stl" />
       </geometry>
       <material name="black"/>
@@ -34,5 +34,5 @@
       <!--<geometry>-->
         <!--<mesh-->
-          <!--filename="package://jetrover_description/meshes/common/lidar_link.stl" />-->
+          <!--filename="$(find jetrover_description)/meshes/common/lidar_link.stl" />-->
       <!--</geometry>-->
     <!--</collision>-->
